File: hardware/pcb/Camera.kicad_sch (KiCad schematic)
At the start: 9 parts, among them U1 SeeeduinoXIAORP2040

Commit message: Fix transistor orientation
Parts:
- n-Mosfet1: value 2N7000 -> 2N7002; footprint Package_TO_SOT_SMD:SOT-23_Handsoldering -> Package_TO_SOT_SMD:SOT-23; symbol Transistor_FET:2N7000 -> Transistor_FET:2N7002
Connections:
- net at 3.3V_reg1.1 (GND), C1.1, C2.1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: now also n-Mosfet1.2 (S); no longer n-Mosfet1.1 (S)
- net at U1.7 (PB08_A6_D6_TX): now also n-Mosfet1.1 (G); no longer n-Mosfet1.2 (G)
Changed lines of the file:
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@@
     (pin "5")
   )
-  (symbol (lib_id "Transistor_FET:2N7000") (at 208.28 43.18 90) (unit 1)
+  (symbol (lib_id "Transistor_FET:2N7002") (at 208.28 43.18 90) (unit 1)
     (in_bom yes) (on_board yes)
     (property "Reference" "n-Mosfet1" (id 0) (at 208.28 34.4932 90))
-    (property "Value" "2N7000" (id 1) (at 208.28 36.8046 90))
-    (property "Footprint" "Package_TO_SOT_SMD:SOT-23_Handsoldering" (id 2) (at 210.185 38.1 0)
+    (property "Value" "2N7002" (id 1) (at 208.28 36.8046 90))
+    (property "Footprint" "Package_TO_SOT_SMD:SOT-23" (id 2) (at 210.185 38.1 0)
       (effects (font (size 1.27 1.27) italic) (justify left) hide)
     )
@@
     )
     (path "/00000000-0000-0000-0000-000061bfb588"
-      (reference "n-Mosfet1") (unit 1) (value "2N7000") (footprint "Package_TO_SOT_SMD:SOT-23_Handsoldering")
+      (reference "n-Mosfet1") (unit 1) (value "2N7002") (footprint "Package_TO_SOT_SMD:SOT-23")
     )
   )
